Commit message: a lot of bugs

File: wrs_gazebo/mobile_dual_arm/urdf/mobile_dual_arm.xacro (robot description, xacro)
@@ -55,52 +55,4 @@
     <child link="Arm_Base_R"/>
   </joint-->
-  <link name="Bin">
-    <inertial>
-      <origin
-	xyz="0 0 0"
-	rpy="0 0 0" />
-      <mass
-	value="0.823603974032196" />
-      <inertia
-	ixx="0"
-	ixy="0"
-	ixz="0"
-	iyy="0"
-	iyz="0"
-	izz="0" />
-    </inertial>
-    <visual>
-      <origin
-	xyz="0 0 0"
-	rpy="0 0 0" />
-      <geometry>
-	<mesh
-          scale="0.001 0.001 0.001"
-	  filename="package://mobile_dual_arm/scene/meshes/bin.STL" />
-      </geometry>
-      <material
-	name="blue_">
-	<color
-	  rgba="0.4 0.66 0.99 1" />
-      </material>
-    </visual>
-    <collision>
-      <origin
-	xyz="0 0 0"
-	rpy="0 0 0" />
-      <geometry>
-	<mesh
-          scale="0.001 0.001 0.001"
-	  filename="package://mobile_dual_arm/scene/meshes/bin.STL" />
-      </geometry>
-    </collision>
-  </link>
-  <joint name="fixed4" type="fixed">
-    <origin
-      xyz="-0.175 -0.31 0.06"
-      rpy="0 0 1.5708" />
-    <parent link="mobile_base"/>
-    <child link="Bin"/>
-  </joint>
   <transmission name="tran1_slide_R">
     <type>transmission_interface/SimpleTransmission</type>

File: wrs_gazebo/mobile_dual_arm/worlds/obj2.urdf (robot description, URDF)
Before this commit: robot obj2, 4 links, 3 joints
Links:
- removed link drink
- removed link lunchbox
- removed link riceball
- removed link sandwich
- added link /right_arm; visual sphere 
Joints:
- removed joint a
- removed joint b
- removed joint c

File: wrs_gazebo/single_arm/single_arm_description/urdf/single_arm.xacro (robot description, xacro)
@@ -107,5 +107,5 @@
 	      upper="3.14"
 	      effort="75"
-	      velocity="65" />
+	      velocity="650" />
 	  </joint>
 	  <link
@@ -165,5 +165,5 @@
 	      upper="3.14"
 	      effort="75"
-	      velocity="65" />
+	      velocity="650" />
 	  </joint>
 	  <link
@@ -223,5 +223,5 @@
 	      upper="3.14"
 	      effort="65"
-	      velocity="65" />
+	      velocity="650" />
 	  </joint>
 	  <link
@@ -281,5 +281,5 @@
 	      upper="3.14"
 	      effort="65"
-	      velocity="65" />
+	      velocity="650" />
 	  </joint>
 	  <link
@@ -339,5 +339,5 @@
 	      upper="3.14"
 	      effort="65"
-	      velocity="65" />
+	      velocity="650" />
 	  </joint>
 	  <link
@@ -397,5 +397,5 @@
 	      upper="3.14"
 	      effort="65"
-	      velocity="65" />
+	      velocity="650" />
 	  </joint>
 	  <!-- <link
@@ -455,5 +455,5 @@
 				upper="3.14"
 				effort="22"
-				velocity="65" />
+				velocity="650" />
 		</joint>
           <!--

Commit message: change kinematics

File: wrs_gazebo/mobile_dual_arm/urdf/mobile_dual_arm.xacro (robot description, xacro)
@@ -23,5 +23,5 @@
   </joint>
   <xacro:single_arm side="r"  parent="Arm_Base_R_Link" child="r_tool_link" toolrot="1.57">
-    <origin xyz="0 -0.016 0" rpy="1.57 1.57 0" />
+    <origin xyz="0 -0.1 0" rpy="1.57 3.14 0" />
   </xacro:single_arm>
   <xacro:suction side="r"  parent="r_Link_6">
@@ -29,5 +29,5 @@
   </xacro:suction>
   <xacro:single_arm side="l"  parent="Arm_Base_L_Link" child="l_tool_link" toolrot="-1.57">
-    <origin xyz="0 0.016 0" rpy="-1.57 1.57 0" />
+    <origin xyz="0 0.1 0" rpy="-1.57 0 0" />
   </xacro:single_arm>
   <xacro:suction side="l"  parent="l_Link_6">

File: wrs_gazebo/single_arm/single_arm_description_old/urdf/single_arm.xacro (robot description, xacro)
@@ -10,5 +10,5 @@
 	    <inertial>
 	      <origin
-		xyz="0.000156250860732315 0.000202963757501797 -0.0546720420122521"
+		xyz="4.11470055452497E-06 -0.000230371464482181 0.0621924893349088"
 		rpy="0 0 0" />
 	      <mass
@@ -55,5 +55,5 @@
 	    <inertial>
 	      <origin
-		xyz="-3.64540734812575E-06 0.00119778550610652 -0.000421399675048756"
+		xyz="0.000398625697734733 -3.44839622274201E-06 0.157268979305323"
 		rpy="0 0 0" />
 	      <mass
@@ -95,6 +95,6 @@
 	    type="revolute">
 	    <origin
-	      xyz="0 0 0.0550000000000002"
-	      rpy="-1.5707963267949 -2.60398896659329E-32 1.5707963267949" />
+	      xyz="0 0 0"
+	      rpy="0 0 -1.5708" />
 	    <parent
 	      link="${side}_Base" />
@@ -102,10 +102,10 @@
 	      link="${side}_Link_1" />
 	    <axis
-	      xyz="0 -1 0" />
+	      xyz="0 0 1" />
 	    <limit
 	      lower="-3.14"
 	      upper="3.14"
 	      effort="75"
-	      velocity="650" />
+	      velocity="65" />
 	  </joint>
 	  <link
@@ -113,5 +113,5 @@
 	    <inertial>
 	      <origin
-		xyz="0.000683310419598862 -8.00535195483731E-05 0.117541995924546"
+		xyz="0.0872199190349209 -2.17078867403853E-06 -0.00123755630277769"
 		rpy="0 0 0" />
 	      <mass
@@ -153,6 +153,6 @@
 	    type="revolute">
 	    <origin
-	      xyz="0 0 0"
-	      rpy="-1.5707963267949 7.39557098644699E-32 -1.5707963267949" />
+	      xyz="0 0 0.16"
+	      rpy="1.5708 0 1.5708" />
 	    <parent
 	      link="${side}_Link_1" />
@@ -160,10 +160,10 @@
 	      link="${side}_Link_2" />
 	    <axis
-	      xyz="0 -1 0" />
+	      xyz="0 0 -1" />
 	    <limit
 	      lower="-3.14"
 	      upper="3.14"
 	      effort="75"
-	      velocity="650" />
+	      velocity="65" />
 	  </joint>
 	  <link
@@ -171,5 +171,5 @@
 	    <inertial>
 	      <origin
-		xyz="-0.0220564838621471 0.101455973505417 -8.62457453022769E-05"
+		xyz="-0.0149070189110112 5.93125910155643E-05 0.262650975551228"
 		rpy="0 0 0" />
 	      <mass
@@ -211,6 +211,6 @@
 	    type="revolute">
 	    <origin
-	      xyz="0 0 0.174"
-	      rpy="1.5707963267949 4.63843178081015E-17 6.91111242388425E-16" />
+	      xyz="0 0 0"
+	      rpy="1.5708 0 1.5708" />
 	    <parent
 	      link="${side}_Link_2" />
@@ -218,10 +218,10 @@
 	      link="${side}_Link_3" />
 	    <axis
-	      xyz="0 1 0" />
+	      xyz="0 0 1" />
 	    <limit
 	      lower="-3.14"
 	      upper="3.14"
 	      effort="65"
-	      velocity="650" />
+	      velocity="65" />
 	  </joint>
 	  <link
@@ -229,5 +229,5 @@
 	    <inertial>
 	      <origin
-		xyz="0.0297389855299131 0.0361651889050357 0.108377256276242"
+		xyz="-0.0294457805062883 -0.0888739607940883 8.91006395364796E-05"
 		rpy="0 0 0" />
 	      <mass
@@ -269,6 +269,6 @@
 	    type="revolute">
 	    <origin
-	      xyz="-0.0299999998727122 0.115999993001519 0.0359999999999999"
-	      rpy="-1.5707963267949 -1.40443212615082E-14 1.75438367537121E-15" />
+	      xyz="-0.03 0 0.29"
+	      rpy="-1.5708 0 -3.1416" />
 	    <parent
 	      link="${side}_Link_3" />
@@ -276,10 +276,10 @@
 	      link="${side}_Link_4" />
 	    <axis
-	      xyz="0 -1 0" />
+	      xyz="0 0 1" />
 	    <limit
 	      lower="-3.14"
 	      upper="3.14"
 	      effort="65"
-	      velocity="650" />
+	      velocity="65" />
 	  </joint>
 	  <link
@@ -287,5 +287,5 @@
 	    <inertial>
 	      <origin
-		xyz="-0.000172095429412281 0.102690028206534 -6.66794215013755E-05"
+		xyz="1.27279603523434E-10 5.99983513058479E-05 0.247701821537204"
 		rpy="0 0 0" />
 	      <mass
@@ -327,6 +327,6 @@
 	    type="revolute">
 	    <origin
-	      xyz="0.029999999872713 0.0359999999999987 0.162"
-	      rpy="1.5707963267949 -8.80083043478898E-16 -2.49800180540655E-16" />
+	      xyz="-0.03 0 0"
+	      rpy="-1.5708 -6.5485E-17 -3.1416" />
 	    <parent
 	      link="${side}_Link_4" />
@@ -334,10 +334,10 @@
 	      link="${side}_Link_5" />
 	    <axis
-	      xyz="0 1 0" />
+	      xyz="0 0 1" />
 	    <limit
 	      lower="-3.14"
 	      upper="3.14"
 	      effort="65"
-	      velocity="650" />
+	      velocity="65" />
 	  </joint>
 	  <link
@@ -345,5 +345,5 @@
 	    <inertial>
 	      <origin
-		xyz="1.14707347786958E-08 0.0359051244401507 0.076720238383497"
+		xyz="1.27298144247945E-10 -0.0744505668165777 -7.66617635603494E-05"
 		rpy="0 0 0" />
 	      <mass
@@ -355,5 +355,5 @@
 		iyy="0.000143902079306418"
 		iyz="2.7663385335139E-07"
-		izz="0.000196835999327886"/>
+		izz="0.000196835999327886" />
 	    </inertial>
 	    <visual>
@@ -385,6 +385,6 @@
 	    type="revolute">
 	    <origin
-	      xyz="0 0.108000511190835 0.0360000000000014"
-	      rpy="-1.5707963267949 0 4.46815747097797E-32" />
+	      xyz="0 0 0.263"
+	      rpy="-1.5708 0 4.5659E-16" />
 	    <parent
 	      link="${side}_Link_5" />
@@ -392,10 +392,10 @@
 	      link="${side}_Link_6" />
 	    <axis
-	      xyz="0 -1 0" />
+	      xyz="0 0 -1" />
 	    <limit
 	      lower="-3.14"
 	      upper="3.14"
 	      effort="65"
-	      velocity="650" />
+	      velocity="65" />
 	  </joint>
 	  <!-- <link
@@ -443,9 +443,6 @@
 			type="revolute">
 			<origin
-				xyz="0 0.03680 0.135"
-				rpy="0 0 0" />
-				<!-- rpy="1.5708 ${toolrot} 0" /> -->
-				<!-- xyz="-0.008041 0.038 0.13545" -->
-				<!-- xyz="-0.0025 0.038 0.135" -->
+				xyz="0 -0.1345 0"
+				rpy="1.5708 ${toolrot} 0" />
 			<parent
 				link="${side}_Link_6" />
@@ -458,5 +455,5 @@
 				upper="3.14"
 				effort="22"
-				velocity="650" />
+				velocity="65" />
 		</joint>
           <!--
