Commit message: final

File: wrs_gazebo/suction_urdf/urdf/suction.gazebo.xacro (robot description, xacro)
@@ -13,5 +13,5 @@
     <mu1>0.2</mu1>
     <mu2>0.2</mu2>
-    <material>Gazebo/white</material>
+    <material>Gazebo/BlackTransparent</material>
     <selfCollide>false</selfCollide>
   </gazebo>
@@ -19,5 +19,5 @@
     <mu1>0.2</mu1>
     <mu2>0.2</mu2>
-    <material>Gazebo/grey</material>
+    <material>Gazebo/BlackTransparent</material>
     <selfCollide>false</selfCollide>
   </gazebo>

File: wrs_gazebo/suction_urdf/urdf/suction_urdf.xacro (robot description, xacro)
@@ -124,5 +124,5 @@
           rpy="0 0 0" />
 	<geometry>
-           <box size="0.01 0.01 0.01"/>
+           <box size="0.001 0.001 0.001"/>
         </geometry>
         <material
@@ -170,5 +170,5 @@
           rpy="0 0 0" />
 	<geometry>
-           <box size="0.01 0.01 0.01"/>
+           <box size="0.001 0.001 0.001"/>
         </geometry>
         <material
@@ -216,5 +216,5 @@
           rpy="0 0 0" />
 	<geometry>
-           <box size="0.01 0.01 0.01"/>
+           <box size="0.001 0.001 0.001"/>
         </geometry>
         <material
@@ -262,5 +262,5 @@
           rpy="0 0 0" />
 	<geometry>
-           <box size="0.01 0.01 0.01"/>
+           <box size="0.001 0.001 0.001"/>
         </geometry>
         <material
@@ -308,5 +308,5 @@
           rpy="0 0 0" />
 	<geometry>
-           <box size="0.01 0.01 0.01"/>
+           <box size="0.001 0.001 0.001"/>
         </geometry>
         <material
